Commit message: inspire hand tip

File: robots/unitree_g1/g1_29dof_rev_1_0_with_inspire_hand_DFQ.urdf (robot description, URDF)
Before this commit: robot g1_29dof_rev_1_0_with_inspire_hand_DFQ, 63 links, 62 joints
Links:
- added link L_index_tip; visual sphere radius=0.005
- added link L_middle_tip; visual sphere radius=0.005
- added link L_pinky_tip; visual sphere radius=0.005
- added link L_ring_tip; visual sphere radius=0.005
- added link L_thumb_tip; visual sphere radius=0.005
- added link R_index_tip; visual sphere radius=0.005
- added link R_middle_tip; visual sphere radius=0.005
- added link R_pinky_tip; visual sphere radius=0.005
- added link R_ring_tip; visual sphere radius=0.005
- added link R_thumb_tip; visual sphere radius=0.005
Joints:
- added joint L_index_tip_joint: type fixed, parent L_index_intermediate, child L_index_tip, origin xyz=-0.00412053 -0.0433132 -0.00501047 rpy=0 0 0
- added joint L_middle_tip_joint: type fixed, parent L_middle_intermediate, child L_middle_tip, origin xyz=-0.00426879 -0.0466043 -0.00498678 rpy=0 0 0
- added joint L_pinky_tip_joint: type fixed, parent L_pinky_intermediate, child L_pinky_tip, origin xyz=-0.00260734 -0.0362776 -0.00501047 rpy=0 0 0
- added joint L_ring_tip_joint: type fixed, parent L_ring_intermediate, child L_ring_tip, origin xyz=-0.00366554 -0.0433541 -0.00501047 rpy=0 0 0
- added joint L_thumb_tip_joint: type fixed, parent L_thumb_distal, child L_thumb_tip, origin xyz=0.0159104 -0.0156076 -0.00599021 rpy=0 0 0
- added joint R_index_tip_joint: type fixed, parent R_index_intermediate, child R_index_tip, origin xyz=-0.00412053 0.0433132 -0.00501047 rpy=0 0 0
- added joint R_middle_tip_joint: type fixed, parent R_middle_intermediate, child R_middle_tip, origin xyz=-0.00426879 0.0466043 -0.00498678 rpy=0 0 0
- added joint R_pinky_tip_joint: type fixed, parent R_pinky_intermediate, child R_pinky_tip, origin xyz=-0.00260734 0.0362776 -0.00501047 rpy=0 0 0
- added joint R_ring_tip_joint: type fixed, parent R_ring_intermediate, child R_ring_tip, origin xyz=-0.00366554 0.0433541 -0.00501047 rpy=0 0 0
- added joint R_thumb_tip_joint: type fixed, parent R_thumb_distal, child R_thumb_tip, origin xyz=0.0159104 0.0156076 -0.00599021 rpy=0 0 0
